File: Smart-halytin.kicad_pcb (KiCad board)
At the start: 2 copper layers, 34 parts, among them J1 Barrel_Jack, SW1 SW_Push, U1 LPC1113FBD48-302, U2 TPS56339DDC, U3 NHD-C0220BIZ, U5 ESP-07, U6 RN4871, U7 TPS56339DDC

Commit message: pcb done
Parts:
- added U4: AMG8854, footprints:AMG8854, F.Cu at (149.9, 87.6)
- added U8: EKMC1607111, footprints:EKMC1607111, F.Cu at (116.8, 100.3)
- moved D1 67.6 mm to (118.1, 74.9), turned to 270 degrees
- moved R11 65.6 mm to (118.1, 78.7), turned to 270 degrees
- moved R12 46.2 mm to (142.2, 101.6)
- moved U5 40.4 mm to (154.9, 69.8), turned to 0 degrees
- moved R1 40.2 mm to (143.5, 87.6), turned to 180 degrees
- moved R3 40.0 mm to (143.5, 85.1), turned to 180 degrees
- moved J1 39.9 mm to (99.1, 85.1)
- moved L1 39.9 mm to (116.8, 81.3)
- moved C5 39.9 mm to (104.6, 87.6)
- moved R6 39.9 mm to (116.8, 95.2)
- moved R7 39.9 mm to (116.8, 86.4)
- moved C10 39.9 mm to (107.5, 88.9)
- moved C4 39.9 mm to (104.1, 94.0)
- moved C6 39.9 mm to (104.6, 83.8)
- moved R10 39.9 mm to (109.2, 97.8)
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Routing:
- net +5V: track 10.7 -> 109.2 mm, vias 2 -> 5
- net GND: track 20.3 -> 95.6 mm, vias 0 -> 8
- net SPI_CS_WIFI: track 0.00 -> 75.0 mm, vias 0 -> 2
- net SCL: track 0.00 -> 72.7 mm, vias 0 -> 4
- net SDA: track 0.00 -> 70.0 mm, vias 0 -> 3
- net +3V3: track 18.0 -> 82.5 mm, vias 3 -> 6
- net LCD_RST: track 0.00 -> 40.5 mm, vias 0 -> 2
- net SPI_CLK: track 0.00 -> 34.7 mm
- net BUTTON_GPIO: track 0.00 -> 33.1 mm, vias 0 -> 2
- net SPI_MOSI: track 0.00 -> 32.9 mm
- net WIFI_RST: track 0.00 -> 32.6 mm, vias 0 -> 2
- net SPI_MISO: track 0.00 -> 22.4 mm
- net Grid-EYE_INT: track 0.00 -> 19.2 mm, vias 0 -> 2
- net LED_GPIO: track 0.00 -> 12.4 mm, vias 0 -> 2
- net PIR_GPIO: track 0.00 -> 12.3 mm
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
Commit message: pcb
Parts:
- moved U6 1.27 mm to (125.7, 72.4)
- moved U3 1.27 mm to (138.4, 134.6)
Connections:
- C3 pad 1: +5V -> +3V3
- R1 pad 2: +5V -> +3V3
- R2 pad 2: +5V -> +3V3
- R3 pad 2: +5V -> +3V3
- U1 pad 23: Net-(U1-Pad23) -> BLE_UART_CTS
- U1 pad 45: Net-(U1-Pad45) -> BLE_UART_RTS
- U1 pad 9: Net-(U1-Pad9) -> BLE_UART_TX_IND
- U4 pad 13: +5V -> +3V3
- U4 pad 9: +5V -> +3V3
- U6 pad 11: Net-(U6-Pad11) -> BLE_UART_CTS
- U6 pad 15: Net-(U6-Pad15) -> BLE_UART_TX_IND
- U6 pad 9: Net-(U6-Pad9) -> BLE_UART_RTS
Routing:
- net BLE_UART_TX_IND: track 0.00 -> 46.1 mm, vias 0 -> 2
- net BLE_UART_CTS: track 0.00 -> 35.3 mm, vias 0 -> 4
- net +3V3: track 82.5 -> 116.0 mm
- net +5V: track 109.2 -> 76.2 mm
- net BLE_UART_RTS: track 0.00 -> 16.7 mm, vias 0 -> 2
- net SPI_CLK: track 34.7 -> 46.2 mm, vias 0 -> 2
- net SPI_CS_WIFI: track 75.0 -> 76.4 mm
- net BLE_RST: track 4.24 -> 5.60 mm
- net SDA: track 70.0 -> 68.7 mm
- net SCL: track 72.7 -> 71.5 mm
- net LCD_RST: track 40.5 -> 39.2 mm
- net BLE_UART_TX: track 6.03 -> 7.30 mm
- net BLE_UART_RX: track 4.24 -> 5.51 mm
- net GND: track 95.6 -> 95.7 mm, vias 8 -> 10

Commit message: lcd connector
Parts:
- removed U3: NHD-C0220BIZ, Display:NHD-C0220BiZ
- added J2: Conn_01x05_Male_LCD_DISPLAY, Connector_JST:JST_VH_B5P-VH-FB-B_1x05_P3.96mm_Vertical, F.Cu at (141.3, 119.4)
Routing:
- net SDA: track 68.7 -> 72.1 mm
- net LCD_RST: track 39.2 -> 41.5 mm
- net SCL: track 71.5 -> 73.2 mm
- net GND: track 95.7 -> 96.4 mm, vias 10 -> 8
